Commit message: added DAE files, and edited urdf to include them. Upadated URDF to contain all links
Still needs joints added

File: src/ik_interface/urdf/rover_arm.urdf (robot description, URDF)
Before this commit: robot rover_arm, 2 links, 1 joints
Links:
- added link arm_hand; collision mesh filename=package://ik_interface/urdf/stl_files/arm_hand.stl; visual mesh filename=package://ik_interface/urdf/dae_files/arm_hand.dae
- added link arm_link_1; collision mesh filename=package://ik_interface/urdf/stl_files/arm_link_1.stl; visual mesh filename=package://ik_interface/urdf/dae_files/arm_link_1.dae
- added link arm_link_2; collision mesh filename=package://ik_interface/urdf/stl_files/arm_link_2.stl; visual mesh filename=package://ik_interface/urdf/dae_files/arm_link_2.dae
- added link arm_link_3; collision mesh filename=package://ik_interface/urdf/stl_files/arm_link_3.stl; visual mesh filename=package://ik_interface/urdf/dae_files/arm_link_3.dae
- added link arm_link_4; collision mesh filename=package://ik_interface/urdf/stl_files/arm_link_4.stl; visual mesh filename=package://ik_interface/urdf/dae_files/arm_link_4.dae
- link arm_link_0: geometry collision mesh filename=package://ik_interface/urdf/stl_files/arm_link_0.stl; visual mesh filename=package://ik_interface/urdf/dae_files/arm_link_0.dae
- link base_link: geometry collision mesh filename=package://ik_interface/urdf/stl_files/base_link.stl; visual mesh filename=package://ik_interface/urdf/dae_files/base_link.dae

Commit message: Added joints to URDF, but needs renaming

File: src/ik_interface/urdf/rover_arm.urdf (robot description, URDF)
Before this commit: robot rover_arm, 7 links, 1 joints
Joints:
- removed joint base_to_link_0
- added joint joint_1: type revolute, parent base_link, child link_1, origin xyz=0 0 0.061584 rpy=0 0 0, axis 0 0 1, limit lower=-3.141592653589793 upper=3.141592653589793 effort=1000.0 velocity=2.5

Commit message: Commented out extra URDF joints and segments
I figure its probably best to work one by one

File: src/ik_interface/urdf/rover_arm.urdf (robot description, URDF)
Before this commit: robot rover_arm, 7 links, 1 joints
Links:
- removed link arm_hand
- removed link arm_link_1
- removed link arm_link_2
- removed link arm_link_3
- removed link arm_link_4

Commit message: added inertial

File: src/ik_interface/urdf/rover_arm.urdf (robot description, URDF)
Before this commit: robot rover_arm, 2 links, 1 joints
Links:
- removed link arm_link_0
- link base_link: mass None -> 1
Joints:
- removed joint joint_1

Commit message: added first 4 joints in urdf

File: src/ik_interface/urdf/rover_arm.urdf (robot description, URDF)
Before this commit: robot rover_arm, 1 links, 0 joints
Links:
- added link arm_link_0, mass 1; collision mesh filename=package://ik_interface/urdf/stl_files/arm_link_0.stl; visual mesh filename=package://ik_interface/urdf/dae_files/arm_link_0.dae
- added link arm_link_1, mass 1; collision mesh filename=package://ik_interface/urdf/stl_files/arm_link_1.stl; visual mesh filename=package://ik_interface/urdf/dae_files/arm_link_1.dae
- added link arm_link_2, mass 1; collision mesh filename=package://ik_interface/urdf/stl_files/arm_link_2.stl; visual mesh filename=package://ik_interface/urdf/dae_files/arm_link_2.dae
- added link arm_link_3, mass 1; collision mesh filename=package://ik_interface/urdf/stl_files/arm_link_3.stl; visual mesh filename=package://ik_interface/urdf/dae_files/arm_link_3.dae
Joints:
- added joint base_joint: type revolute, parent base_link, child arm_link_0, origin xyz=0 0.055 0.087245 rpy=0 0 0, axis 0 0 1, limit lower=-3.141592653589793 upper=3.141592653589793 effort=1000.0 velocity=2.5
- added joint elbow_pitch_joint: type revolute, parent arm_link_1, child arm_link_2, origin xyz=0.05925 0 0.501983 rpy=0 0 0, axis 1 0 0, limit lower=-3.141592653589793 upper=3.141592653589793 effort=1000.0 velocity=2.5
- added joint elbow_roll_joint: type revolute, parent arm_link_2, child arm_link_3, origin xyz=0.063 0.000654 0.059505 rpy=0 0 0, axis 0 0 1, limit lower=-3.141592653589793 upper=3.141592653589793 effort=1000.0 velocity=2.5
- added joint shoulder_joint: type revolute, parent arm_link_0, child arm_link_1, origin xyz=0 0 0.151443 rpy=0 0 0, axis 1 0 0, limit lower=-3.141592653589793 upper=3.141592653589793 effort=1000.0 velocity=2.5

Commit message: Added final two joints and segments to URDF

File: src/ik_interface/urdf/rover_arm.urdf (robot description, URDF)
Before this commit: robot rover_arm, 5 links, 4 joints
Links:
- added link arm_gripper, mass 1; collision mesh filename=package://ik_interface/urdf/stl_files/arm_gripper.stl; visual mesh filename=package://ik_interface/urdf/dae_files/arm_gripper.dae
- added link arm_link_4, mass 1; collision mesh filename=package://ik_interface/urdf/stl_files/arm_link_4.stl; visual mesh filename=package://ik_interface/urdf/dae_files/arm_link_4.dae
Joints:
- added joint gripper_joint: type revolute, parent arm_link_4, child arm_gripper, origin xyz=-0.050 0 0.050484 rpy=0 0 0, axis 0 0 1, limit lower=-3.141592653589793 upper=3.141592653589793 effort=1000.0 velocity=2.5
- added joint wrist_pitch_joint: type revolute, parent arm_link_3, child arm_link_4, origin xyz=-0.065 0 0.3318 rpy=0 0 0, axis 1 0 0, limit lower=-3.141592653589793 upper=3.141592653589793 effort=1000.0 velocity=2.5

Commit message: added joint limits and fixed collision coordinates

File: src/ik_interface/urdf/rover_arm.urdf (robot description, URDF)
Before this commit: robot rover_arm, 7 links, 6 joints
Joints:
- joint base_joint: limit lower=-3.141592653589793 upper=3.141592653589793 effort=1000.0 velocity=2.5 -> lower=-1.57079632679 upper=1.57079632679 effort=1000.0 velocity=2.5
- joint elbow_pitch_joint: limit lower=-3.141592653589793 upper=3.141592653589793 effort=1000.0 velocity=2.5 -> lower=-1.57079632679 upper=1.57079632679 effort=1000.0 velocity=2.5
- joint gripper_joint: limit lower=-3.141592653589793 upper=3.141592653589793 effort=1000.0 velocity=2.5 -> effort=1000.0 velocity=2.5; type revolute -> continuous
- joint shoulder_joint: limit lower=-3.141592653589793 upper=3.141592653589793 effort=1000.0 velocity=2.5 -> lower=-1.57079632679 upper=1.57079632679 effort=1000.0 velocity=2.5
- joint wrist_pitch_joint: limit lower=-3.141592653589793 upper=3.141592653589793 effort=1000.0 velocity=2.5 -> lower=-1.57079632679 upper=3.141592653589793 effort=1000.0 velocity=2.5
