Commit message: renamed gripper_joint to wrist_roll_joint

File: src/rover_arm/config/rover_arm.ros2_control.xacro (robot description, xacro)
@@ -2,14 +2,16 @@
 <robot xmlns:xacro="http://www.ros.org/wiki/xacro">
     <xacro:macro name="rover_arm_ros2_control" params="name initial_positions_file">
-        <xacro:property name="initial_positions" value="${load_yaml(initial_positions_file)['initial_positions']}"/>
+        <xacro:property name="initial_positions" value="${xacro.load_yaml(initial_positions_file)['initial_positions']}"/>
         <ros2_control name="${name}" type="system">
             <hardware>
-                <!-- By default, set up controllers for simulation. This won't work on real hardware -->
+                <!-- <plugin>odrive_ros2_control_plugin/ODriveHardwareInterface</plugin> -->
+                <!-- <param name="can">can0</param> -->
                 <plugin>mock_components/GenericSystem</plugin>
             </hardware>
             <joint name="base_joint">
+                <param name="node_id">0</param>
+                <param name="gear_ratio">400.0</param>
                 <command_interface name="position"/>
                 <command_interface name="velocity"/>
-                <command_interface name="effort"/>
                 <state_interface name="position">
                   <param name="initial_value">${initial_positions['base_joint']}</param>
@@ -19,7 +21,8 @@
             </joint>
             <joint name="shoulder_joint">
+                <param name="node_id">1</param>
+                <param name="gear_ratio">640.0</param>
                 <command_interface name="position"/>
                 <command_interface name="velocity"/>
-                <command_interface name="effort"/>
                 <state_interface name="position">
                   <param name="initial_value">${initial_positions['shoulder_joint']}</param>
@@ -29,7 +32,8 @@
             </joint>
             <joint name="elbow_pitch_joint">
+                <param name="node_id">2</param>
+                <param name="gear_ratio">420.0</param>
                 <command_interface name="position"/>
                 <command_interface name="velocity"/>
-                <command_interface name="effort"/>
                 <state_interface name="position">
                   <param name="initial_value">${initial_positions['elbow_pitch_joint']}</param>
@@ -39,7 +43,8 @@
             </joint>
             <joint name="elbow_roll_joint">
+                <param name="node_id">3</param>
+                <param name="gear_ratio">120.0</param>
                 <command_interface name="position"/>
                 <command_interface name="velocity"/>
-                <command_interface name="effort"/>
                 <state_interface name="position">
                   <param name="initial_value">${initial_positions['elbow_roll_joint']}</param>
@@ -49,7 +54,8 @@
             </joint>
             <joint name="wrist_pitch_joint">
+                <param name="node_id">4</param>
+                <param name="gear_ratio">300.0</param>
                 <command_interface name="position"/>
                 <command_interface name="velocity"/>
-                <command_interface name="effort"/>
                 <state_interface name="position">
                   <param name="initial_value">${initial_positions['wrist_pitch_joint']}</param>
@@ -58,10 +64,11 @@
                 <state_interface name="effort"/>
             </joint>
-            <joint name="gripper_joint">
+            <joint name="wrist_roll_joint">
+                <param name="node_id">5</param>
+                <param name="gear_ratio">1.0</param>
                 <command_interface name="position"/>
                 <command_interface name="velocity"/>
-                <command_interface name="effort"/>
                 <state_interface name="position">
-                  <param name="initial_value">${initial_positions['gripper_joint']}</param>
+                  <param name="initial_value">${initial_positions['wrist_roll_joint']}</param>
                 </state_interface>
                 <state_interface name="velocity"/>

File: src/rover_arm_urdf/urdf/rover_arm.urdf (robot description, URDF)
Before this commit: robot rover_arm, 7 links, 6 joints
Joints:
- removed joint gripper_joint
- added joint wrist_roll_joint: type continuous, parent arm_link_4, child arm_gripper, origin xyz=-0.050 0 0.050484 rpy=0 0 0, axis 0 0 1, limit effort=1000.0 velocity=2.5
