Commit message: whole lotta changes

File: rover_arm/config/rover_arm.urdf.xacro (robot description, xacro)
@@ -6,4 +6,4 @@
     <!-- Import control_xacro -->
     <xacro:include filename="rover_arm.ros2_control.xacro" />
-    <xacro:rover_arm_ros2_control name="FakeSystem" initial_positions_file="$(arg initial_positions_file)"/>
+    <xacro:rover_arm_ros2_control name="RealSystem" initial_positions_file="$(arg initial_positions_file)"/>
 </robot>

File: rover_arm_urdf/urdf/rover_arm.urdf (robot description, URDF)
Before this commit: robot rover_arm, 7 links, 6 joints
Links:
- link arm_gripper: geometry collision mesh filename=package://rover_arm_urdf/urdf/stl_files/arm_gripper.stl; visual mesh filename=package://rover_arm_urdf/urdf/dae_files/arm_gripper.dae
- link arm_link_0: geometry collision mesh filename=package://rover_arm_urdf/urdf/stl_files/arm_link_0.stl; visual mesh filename=package://rover_arm_urdf/urdf/dae_files/arm_link_0.dae
- link arm_link_1: geometry collision mesh filename=package://rover_arm_urdf/urdf/stl_files/arm_link_1.stl; visual mesh filename=package://rover_arm_urdf/urdf/dae_files/arm_link_1.dae
- link arm_link_2: geometry collision mesh filename=package://rover_arm_urdf/urdf/stl_files/arm_link_2.stl; visual mesh filename=package://rover_arm_urdf/urdf/dae_files/arm_link_2.dae
- link arm_link_3: geometry collision mesh filename=package://rover_arm_urdf/urdf/stl_files/arm_link_3.stl; visual mesh filename=package://rover_arm_urdf/urdf/dae_files/arm_link_3.dae
- link arm_link_4: geometry collision mesh filename=package://rover_arm_urdf/urdf/stl_files/arm_link_4.stl; visual mesh filename=package://rover_arm_urdf/urdf/dae_files/arm_link_4.dae
- link base_link: mass 1 -> None; geometry collision mesh filename=package://rover_arm_urdf/urdf/stl_files/base_link.stl; visual mesh filename=package://rover_arm_urdf/urdf/dae_files/base_link.dae
