Commit message: fixed elbow pitch

File: rover_arm_urdf/urdf/rover_arm.urdf (robot description, URDF)
Before this commit: robot rover_arm, 7 links, 6 joints
Joints:
- joint elbow_pitch_joint: axis 1 0 0 -> -1 0 0

Commit message: fixed all axis

File: rover_arm_urdf/urdf/rover_arm.urdf (robot description, URDF)
Before this commit: robot rover_arm, 7 links, 6 joints
Joints:
- joint base_joint: axis 0 0 1 -> 0 0 -1
- joint elbow_roll_joint: axis 0 0 1 -> 0 0 -1
- joint shoulder_joint: axis 1 0 0 -> -1 0 0
- joint wrist_pitch_joint: axis 1 0 0 -> -1 0 0
- joint wrist_roll_joint: axis 0 0 1 -> 0 0 -1

Commit message: fixed gripper orientation

File: rover_arm_urdf/urdf/rover_arm.urdf (robot description, URDF)
Before this commit: robot rover_arm, 7 links, 6 joints
Joints:
- joint wrist_roll_joint: axis 0 0 -1 -> 0 0 1

Commit message: increased wrist pitch limits

File: rover_arm_urdf/urdf/rover_arm.urdf (robot description, URDF)
Before this commit: robot rover_arm, 7 links, 6 joints
Joints:
- joint elbow_pitch_joint: limit lower=-1.57079632679 upper=1.57079632679 effort=1000.0 velocity=2.5 -> lower=-1.57079632679 upper=2.61799387799 effort=1000.0 velocity=2.5

Commit message: changed velocity limits

File: rover_arm_urdf/urdf/rover_arm.urdf (robot description, URDF)
Before this commit: robot rover_arm, 7 links, 6 joints
Joints:
- joint base_joint: limit lower=-1.57079632679 upper=1.57079632679 effort=1000.0 velocity=2.5 -> lower=-1.57079632679 upper=1.57079632679 effort=1000.0 velocity=2.0
- joint elbow_pitch_joint: limit lower=-1.57079632679 upper=2.61799387799 effort=1000.0 velocity=2.5 -> lower=-1.57079632679 upper=2.61799387799 effort=1000.0 velocity=2.0
- joint elbow_roll_joint: limit lower=-3.141592653589793 upper=3.141592653589793 effort=1000.0 velocity=2.5 -> lower=-3.141592653589793 upper=3.141592653589793 effort=1000.0 velocity=2.0
- joint shoulder_joint: limit lower=-1.57079632679 upper=1.57079632679 effort=1000.0 velocity=2.5 -> lower=-1.57079632679 upper=1.57079632679 effort=1000.0 velocity=2.0
- joint wrist_pitch_joint: limit lower=-1.57079632679 upper=3.141592653589793 effort=1000.0 velocity=2.5 -> lower=-1.57079632679 upper=3.141592653589793 effort=1000.0 velocity=2.0
- joint wrist_roll_joint: limit effort=1000.0 velocity=2.5 -> effort=1000.0 velocity=2.0
